File: Hardware/Design/16197.brd (EAGLE design)
At the start: 61 x 53.3 mm, 83 parts, among them J1 Pi Zero, J2 JTAG, J3 RJ45J, J4 PBC10SAAN, J5 RJ45J, J6 PBC10SAAN, J7 PBC10SAAN, J8 PBC08SAAN, J9 PPPC032LFBN, Q1 K38, Q2 K38, Q3 K38, U1 3172EIBZ, U2 74LVC07A, U3 3172EIBZ, U4 I50115, U5 3172EIBZ, U6 ATMEGA328P-AU, U7 KB33, Y1 14.7456MHz

Commit message: Hardware: ^2 dsgn in wip
Parts:
- removed J10: (no value), U-AVR:ISP
- added C16: 15pF, C-C:C0603(1608)
- added R35, R44: 10K, R-C:C0805(2012)
- added R36, R37, R43, R45: 1.82k, R-C:C0805(2012)
- added R38, R40: 10k, R-C:C0805(2012)
- added R39: 100k, R-C:C0805(2012)
- added R41, R42: OPEN, R-C:C0805(2012)
- added U8: KB33, P-DCDC:SOT23-5,SOT25
- C10: value 10uF -> .1uF; device C-T:3216 -> C-C:C0603(1608)
- C11: value OPEN -> 470pF; device C-C:C0805(2012) -> C-C:C0603(1608)
- C12: value .1uF -> 10uF; device C-C:C0603(1608) -> C-T:3216
- C13: value 15pF -> 0.1uF
- C14: value 15pF -> .1uF
- C15: value 0.1uF -> 15pF
- C4: value 0.1uF -> .1uF
- C9: value 470pF -> .1uF
- J2: value JTAG -> RJ45J; device U-ARM:JTAG -> J-RJ45:RJ45-8HZT
- J3, J5: value RJ45J -> PBC10SAAN; device J-RJ45:RJ45-8HZT -> J-HDR2.54mm:1X10
- J4: value PBC10SAAN -> RJ45J; device J-HDR2.54mm:1X10 -> J-RJ45:RJ45-8HZT
- J7: value PBC10SAAN -> PBC08SAAN; device J-HDR2.54mm:1X10 -> J-HDR2.54mm:1X8
- J8: value PBC08SAAN -> PPPC032LFBN; device J-HDR2.54mm:1X8 -> J-HDR2.54mm:F2X3
- J9: value PPPC032LFBN -> (none); device J-HDR2.54mm:F2X3 -> U-AVR:ISP
- R1: value JMP -> 10k
- R10, R11, R34: value 1.82k -> 3.01k
- R12: value 100 -> 10K
- R13: value 3.01k -> 100
- R14: value 10k -> OPEN
- R15, R4: value 10k -> 1.82k
- R16: value 100 -> 1.82k
- R17, R26: value 3.01k -> 1.82k
- R18: value 1.82k -> 10K
- R2, R22, R7: value 100 -> 10k
- R20: value 200k -> 100
- R21: value 10k -> 3.01k
- R23, R3: value 3.01k -> 10k
- R25: value 182 -> 3.01k
- R28: value OPEN -> 100k
- R29, R8: value OPEN -> 10k
- R30, R32: value 10k -> 100
- R31: value 100k -> 3.01k
- R33: value 1.82k -> 182
- R6: value 10K -> 3.01k
- R9: value 1.82k -> 100
- U1, U3: value 3172EIBZ -> 74LVC07A; device U-Transceiver:SOIC8 -> U-7400:14SOIC
- U2: value 74LVC07A -> 3172EIBZ; device U-7400:14SOIC -> U-Transceiver:SOIC8
- U4: value I50115 -> 3172EIBZ; device P-DCDC:OKI-78SR-H -> U-Transceiver:SOIC8
- U5: value 3172EIBZ -> I50115; device U-Transceiver:SOIC8 -> P-DCDC:OKI-78SR-H
- U6: value ATMEGA328P-AU -> 3172EIBZ; device U-AVR:TQFP32-08 -> U-Transceiver:SOIC8
- U7: value KB33 -> ATMEGA328P-AU; device P-DCDC:SOT23-5,SOT25 -> U-AVR:TQFP32-08
- Y1: value 14.7456MHz -> 12MHz
- moved J5 62.3 mm to (3.56, 50.8), flipped to the bottom, turned to 180 degrees
- moved J6 57.9 mm to (35.6, 2.54)
- moved R33 52.8 mm to (50.7, 48.9), turned to 180 degrees
- moved R27 51.1 mm to (53.6, 33.3), turned to 90 degrees
- moved R34 47.2 mm to (45.2, 6.73), turned to 270 degrees
- moved R2 45.0 mm to (47.9, 45.5), flipped to the bottom, turned to 270 degrees
- moved R31 43.6 mm to (57.4, 8.64)
- moved J9 43.3 mm to (5.08, 31.8), flipped to the top, turned to 90 degrees
- moved U6 43.2 mm to (54.5, 13.1), turned to 270 degrees
- moved R25 42.1 mm to (32.6, 9.65), turned to 90 degrees
- moved J3 41.2 mm to (53.3, 50.8), flipped to the bottom, turned to 0 degrees
- moved R15 38.3 mm to (31.4, 45.3), turned to 270 degrees
- moved J4 37.5 mm to (53.3, 13.3), flipped to the top, turned to 90 degrees
- moved R9 37.3 mm to (21.6, 8.89), flipped to the top
- moved C12 37.1 mm to (27.2, 4.83), turned to 180 degrees
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Connections:
- removed net 3V3PI: J1.1, J2.4, R1.1, R1.2, R9.1
- removed net IOREF_ADC6: C15.1, R31.1, R32.1, U6.19
- removed net N$3: J8.7, R31.2
- removed net SCL0: J1.5, R29.1, U6.28
- removed net SDA0: J1.3, R28.1, U6.27
- removed net SWDCLK: J1.22, J2.1
- removed net SWDIO: J1.18, J2.5
- removed net TARGET_!RST!: J1.12, J2.6
- removed net VIN_ADC7: C4.1, R20.2, R21.1, U6.22
- new net 5V_ADC6: C13.1, R39.1, R40.1, U7.19
- new net N$1: J1.8, R2.2, U1.5
- new net N$4: J1.11, R1.2, U1.9
- new net N$5: R16.2, R19.2, U3.12
- new net N$6: R17.2, R18.2, U3.10
- new net N$7: R43.1, R44.2, S2.1, S2.2
- new net PI3V3: C6.1, C7.1, J1.1, R1.1, R15.1, R2.1, R28.1, R3.2, R4.2, U1.14, U3.14
- new net PI3V3_ADC7: C8.1, R28.2, R29.1, U7.22
- new net PI_!CTS: J1.36, R3.1, U1.2
- new net PI_RX: J1.10, R4.1, U1.4
- new net PI_SCL: J1.5, R41.1
- new net PI_SDA: J1.3, R42.1
- new net SCL1: R41.2, U7.6
- new net SDA1: R42.2, U7.3
- net !RESET: now also J7.6, U3.8; no longer J8.6, U2.8
- net +3V3: now also C10.1, C12.+, C9.1, J9.2, R12.1, R14.1, R22.2, R23.2, R35.2, R36.2, R37.2, R45.1, R5.2, R6.2, R7.2, R8.2, U2.8, U4.8, U6.8, U7.18, U7.4, U8.5; no longer C10.+, C6.1, C7.1, C8.1, J10.2, R14.2, R15.2, R27.2, R34.1, R4.2, R6.1, R8.1, U1.8, U2.14, U3.8, U5.8, U6.18, U6.4, U7.5
- net +5V: now also U5.3; no longer U4.3
- net +DTR: now also J2.6, J4.6, R20.1, U4.6; no longer J3.6, J5.6, R12.1, U3.6
- net +RX: now also J2.8, J4.8, R30.1, U6.6; no longer J3.8, J5.8, R22.1, U5.6
- net +TX: now also J2.2, J4.2, R9.1, U2.6; no longer J3.2, J5.2, R2.1, U1.6
- net -DTR: now also J2.3, J4.3, R20.2, U4.7; no longer J3.3, J5.3, R12.2, U3.7
- net -RX: now also J2.7, J4.7, R30.2, U6.7; no longer J3.7, J5.7, R22.2, U5.7
- net -TX: now also J2.1, J4.1, R9.2, U2.7; no longer J3.1, J5.1, R2.2, U1.7
- net 0V: now also C10.2, C11.2, C12.-, C16.2, J2.4, J2.5, J4.4, J4.5, J6.9, J7.2, J7.3, J8.6, R10.1, R21.1, R29.2, R31.2, R40.2, U1.11, U1.13, U1.7, U2.5, U3.7, U4.5, U5.2, U7.21, U7.5, U8.2; no longer C10.-, C12.2, J10.6, J2.10, J2.2, J3.4, J3.5, J5.5, J6.4, J7.9, J8.2, J8.3, R13.1, R21.2, R23.2, R3.1, R32.2, U1.5, U2.7, U3.5, U4.2, U5.5, U6.21, U7.2
- net DTR_!RE: now also R21.2, U4.2, U7.10; no longer R13.2, U3.2, U6.10
- net DTR_DE: now also R25.2, U7.11; no longer R17.2, U6.11
- net DTR_RXD: now also R26.2, U7.30; no longer R18.2, U6.30
- net DTR_TXD: now also R24.2, U4.4, U7.31; no longer R16.2, U3.4, U6.31
- net HOST_!CTS: now also R8.1, U1.1, U7.23; no longer J1.36, U6.23
- net HOST_!DSR: now also U7.24; no longer U6.24
- net HOST_!DTR: now also U7.32; no longer U6.32
- net HOST_!RTS: now also R5.1, U1.8, U7.1; no longer C11.1, J1.11, U6.1
- net HOST_MISO: now also R15.2, U3.4; no longer R9.2, U2.4
- net HOST_MOSI: now also U3.11; no longer U2.11
- net HOST_RX: now also R7.1, U1.3, U2.1; no longer J1.10, R4.1, U1.1
- net HOST_SCK: now also U3.13; no longer U2.13
- net HOST_TX: now also R32.1, R6.1, U1.6, U6.4; no longer J1.8, R24.1, U5.4
- net ICP1: now also R43.2, U7.12; no longer R33.2, U6.12
- net IOREF: now also J8.2, R16.1, R17.1, R27.1; no longer J9.2, R10.1, R11.1, R19.1
- net LED_BUILTIN: now also U7.13; no longer U6.13
- net MGR_!RESET: now also J9.5, R35.1, U7.29; no longer J10.5, R27.1, U6.29
- net MGR_!SS!: now also R38.1, U7.14; no longer R30.1, U6.14
- net MGR_AREF: now also C14.1, U7.20; no longer C12.1, U6.20
- net MGR_MISO: now also J9.1, U7.16; no longer J10.1, U6.16
- net MGR_MOSI: now also J9.4, U7.15; no longer J10.4, U6.15
- net MGR_SCK: now also J9.3, U7.17; no longer J10.3, U6.17
- net MISO: now also J8.1, U3.3; no longer J9.1, U2.3
- net MOSI: now also J8.4, R18.1; no longer J9.4, R11.2, U2.10
- net N$10: now also R27.2, R33.2, U3.6; no longer R19.2, R25.2, U2.6
- net N$11: now also R34.2, U6.3; no longer R26.2, U5.3
- net N$15: now also R13.1; no longer R7.1
- net N$18: now also R11.1, U2.3; no longer R5.1, U1.3
- net N$19: now also R22.1, R26.1, U4.1; no longer R14.1, R18.1, U3.1
- net N$2: now also R38.2, U3.9; no longer C11.2, R30.2, U2.9
- net N$20: now also R25.1, U4.3; no longer R17.1, U3.3
- net N$22: now also R24.1; no longer R16.1
- net N$24: now also C11.1, U8.4; no longer C9.1, U7.4
- net N$25: now also R32.2; no longer R24.2
- net N$29: now also R45.2; no longer R34.2
- net NODE5V: now also J7.4, R39.2, U8.1, U8.3; no longer J8.4, U7.1, U7.3
- net RX: now also J3.3, R33.1; no longer J4.3, R25.1
- net RX_!RE: now also R31.1, U7.2; no longer R23.1, U5.2
- net RX_DE: now also R34.1, U7.26; no longer R26.1, U6.26
- net RX_RPU: now also R23.1, U3.5, U6.1; no longer R15.1, U2.5, U5.1
- net SCK: now also J8.3, R19.1; no longer J9.3, R10.2, U2.12
- net SCL: now also J5.1, R37.1, U7.28; no longer J6.1, R29.2
- net SDA: now also J5.2, R36.1, U7.27; no longer J6.2, R28.2
- net SHUTDOWN: now also R44.1; no longer R33.1, S2.1, S2.2
- net TX: now also J3.4, R13.2, R14.2, U3.1; no longer J4.4, R7.2, R8.2, U2.1
- net TX_!RE: now also R10.2, U2.2, U7.25; no longer R3.2, U1.2, U6.25
- net TX_DE: now also R11.2, U7.9; no longer R5.2, U6.9
- net TX_RPU: now also R12.2, U2.4, U3.2; no longer R6.2, U1.4, U2.2
- net VIN: now also C4.1, J7.1, U5.1; no longer J8.1, R20.1, U4.1
- net XTAL1: now also C15.1, U7.7; no longer C13.1, U6.7
- net XTAL2: now also C16.1, U7.8; no longer C14.1, U6.8
Routing:
- net DTR_!RE: track 67.8 -> 0.00 mm, vias 4 -> 0
- net +3V3: track 147.8 -> 81.7 mm, vias 13 -> 5
- net RX_DE: track 59.7 -> 0.00 mm, vias 2 -> 0
- net SCL0: track 58.1 -> 0.00 mm, vias 6 -> 0
- net SDA0: track 55.6 -> 0.00 mm, vias 4 -> 0
- net RX_!RE: track 56.0 -> 5.67 mm, vias 2 -> 0
- net DTR_TXD: track 51.8 -> 2.66 mm, vias 2 -> 0
- net DTR_DE: track 48.4 -> 0.00 mm, vias 2 -> 0
- net TX: track 64.2 -> 16.3 mm, vias 6 -> 1
- net HOST_RX: track 46.3 -> 0.00 mm, vias 2 -> 0
- net HOST_MISO: track 45.6 -> 0.00 mm, vias 5 -> 0
- net IOREF_ADC6: track 44.7 -> 0.00 mm, vias 2 -> 0
- net HOST_TX: track 50.8 -> 7.87 mm, vias 2 -> 0
- net VIN_ADC7: track 42.9 -> 0.00 mm, vias 4 -> 0
- net SWDCLK: track 39.1 -> 0.00 mm, vias 2 -> 0
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Other:
- board text added: "16197^2"
- board text added: "HOST !DSR"
- board text added: "HOST !DTR"
- board text added: "RPUBUS.ORG"
- board text removed: "16197^1"
- board text removed: "HOST_!DSR"
- board text removed: "HOST_!DTR"
- board text removed: "SWCLK"
- board text removed: "SWD JTAG"
- board text removed: "SWDIO"
