File: Hardware/Design/16197.sch (EAGLE design)
At the start: 83 parts, among them J1 Pi Zero, J2 JTAG, J3 RJ45J, J4 PBC10SAAN, J5 RJ45J, J6 PBC10SAAN, J7 PBC10SAAN, J8 PBC08SAAN, J9 PPPC032LFBN, Q1 K38, Q2 K38, Q3 K38, U1 3172EIBZ, U2 74LVC07A, U3 3172EIBZ, U4 I50115, U5 3172EIBZ, U6 ATMEGA328P-AU, U7 KB33, Y1 14.7456MHz

Commit message: Hardware: ^2 dsgn in wip
Parts:
- removed J10: (no value), U-AVR:ISP-SPIPTH
- added C16: 15pF, C-C:CC0603A
- added R35, R44: 10K, R-C:R0805
- added R36, R37, R43, R45: 1.82k, R-C:R0805
- added R38, R40: 10k, R-C:R0805
- added R39: 100k, R-C:R0805
- added R41, R42: OPEN, R-C:R0805
- added U8: KB33, P-DCDC:MIC5205
- C10: value 10uF -> .1uF; device C-T:CT1206 -> C-C:CC0603A
- C11: value OPEN -> 470pF; device C-C:CC0805A -> C-C:CC0603A
- C12: value .1uF -> 10uF; device C-C:CC0603A -> C-T:CT1206
- C13: value 15pF -> 0.1uF
- C14: value 15pF -> .1uF
- C15: value 0.1uF -> 15pF
- C4: value 0.1uF -> .1uF
- C9: value 470pF -> .1uF
- J2: value JTAG -> RJ45J; device U-ARM:JTAG_SWD -> J-RJ45:RJ45-8HZT
- J3, J5: value RJ45J -> PBC10SAAN; device J-RJ45:RJ45-8HZT -> J-HDR2.54mm:1X10"
- J4: value PBC10SAAN -> RJ45J; device J-HDR2.54mm:1X10" -> J-RJ45:RJ45-8HZT
- J7: value PBC10SAAN -> PBC08SAAN; device J-HDR2.54mm:1X10" -> J-HDR2.54mm:1X8"
- J8: value PBC08SAAN -> PPPC032LFBN; device J-HDR2.54mm:1X8" -> J-HDR2.54mm:F2X3
- J9: value PPPC032LFBN -> (none); device J-HDR2.54mm:F2X3 -> U-AVR:ISP-SPIPTH
- R1: value JMP -> 10k
- R10, R11, R34: value 1.82k -> 3.01k
- R12: value 100 -> 10K
- R13: value 3.01k -> 100
- R14: value 10k -> OPEN
- R15, R4: value 10k -> 1.82k
- R16: value 100 -> 1.82k
- R17, R26: value 3.01k -> 1.82k
- R18: value 1.82k -> 10K
- R2, R22, R7: value 100 -> 10k
- R20: value 200k -> 100
- R21: value 10k -> 3.01k
- R23, R3: value 3.01k -> 10k
- R25: value 182 -> 3.01k
- R28: value OPEN -> 100k
- R29, R8: value OPEN -> 10k
- R30, R32: value 10k -> 100
- R31: value 100k -> 3.01k
- R33: value 1.82k -> 182
- R6: value 10K -> 3.01k
- R9: value 1.82k -> 100
- U1, U3: value 3172EIBZ -> 74LVC07A; device U-Transceiver:ISL3172EIBZ -> U-7400:7407D
- U2: value 74LVC07A -> 3172EIBZ; device U-7400:7407D -> U-Transceiver:ISL3172EIBZ
- U4: value I50115 -> 3172EIBZ; device P-DCDC:OKI-78SR-H -> U-Transceiver:ISL3172EIBZ
- U5: value 3172EIBZ -> I50115; device U-Transceiver:ISL3172EIBZ -> P-DCDC:OKI-78SR-H
- U6: value ATMEGA328P-AU -> 3172EIBZ; device U-AVR:ATMEGA328PB-AU -> U-Transceiver:ISL3172EIBZ
- U7: value KB33 -> ATMEGA328P-AU; device P-DCDC:MIC5205 -> U-AVR:ATMEGA328PB-AU
- Y1: value 14.7456MHz -> 12MHz
Connections:
- removed net 3V3PI: J1.3V3@1, J2.VCC, R1.1, R1.2, R9.1
- removed net IOREF_ADC6: C15.1, R31.1, R32.1, U6.(ICP3/!SS1!)PE2
- removed net N$3: J8.7, R31.2
- removed net SCL0: J1.BCM3/SCL, R29.1, U6.(A5/SCL0)PC5
- removed net SDA0: J1.BCM2/SDA, R28.1, U6.(A4/SDA0)PC4
- removed net SWDCLK: J1.SD_DAT1/BCM25, J2.TCK:SWDCK
- removed net SWDIO: J1.SD_DAT0/BCM24, J2.TMS:SWDIO
- removed net TARGET_!RST!: J1.!CE10!/BCM18, J2.!RESET
- removed net VIN_ADC7: C4.1, R20.2, R21.1, U6.(A7/T3/MOSI1)PE3
- new net 5V_ADC6: C13.1, R39.1, R40.1, U7.(ICP3/!SS1!)PE2
- new net N$1: J1.TXD/BCM14, R2.2, U1C.I
- new net N$4: J1.BCM17/!CE11!, R1.2, U1D.I
- new net N$5: R16.2, R19.2, U3F.O
- new net N$6: R17.2, R18.2, U3E.O
- new net N$7: R43.1, R44.2, S2.1, S2.2
- new net PI3V3: C6.1, C7.1, J1.3V3@1, R1.1, R15.1, R2.1, R28.1, R3.2, R4.2, U1P.VCC, U3P.VCC
- new net PI3V3_ADC7: C8.1, R28.2, R29.1, U7.(A7/T3/MOSI1)PE3
- new net PI_!CTS: J1.!CE12!/BCM16, R3.1, U1A.O
- new net PI_RX: J1.RXD/BCM15, R4.1, U1B.O
- new net PI_SCL: J1.BCM3/SCL, R41.1
- new net PI_SDA: J1.BCM2/SDA, R42.1
- new net SCL1: R41.2, U7.PE1(SCL1/T4)
- new net SDA1: R42.2, U7.PE0(SDA1/ICP4)
- net !RESET: now also J7.6, U3D.O; no longer J8.6, U2D.O
- net +3V3: now also C10.1, C12.+, C9.1, J9.VCC, R12.1, R14.1, R22.2, R23.2, R35.2, R36.2, R37.2, R45.1, R5.2, R6.2, R7.2, R8.2, U2.VCC, U4.VCC, U6.VCC, U7.AVCC, U7.VCC@0, U8.OUT; no longer C10.+, C6.1, C7.1, C8.1, J10.VCC, R14.2, R15.2, R27.2, R34.1, R4.2, R6.1, R8.1, U1.VCC, U2P.VCC, U3.VCC, U5.VCC, U6.AVCC, U6.VCC@0, U7.OUT
- net +5V: now also U5.VOUT; no longer U4.VOUT
- net +DTR: now also J2.6, J4.6, R20.1, U4.A/Y; no longer J3.6, J5.6, R12.1, U3.A/Y
- net +RX: now also J2.8, J4.8, R30.1, U6.A/Y; no longer J3.8, J5.8, R22.1, U5.A/Y
- net +TX: now also J2.2, J4.2, R9.1, U2.A/Y; no longer J3.2, J5.2, R2.1, U1.A/Y
- net -DTR: now also J2.3, J4.3, R20.2, U4.B/Z; no longer J3.3, J5.3, R12.2, U3.B/Z
- net -RX: now also J2.7, J4.7, R30.2, U6.B/Z; no longer J3.7, J5.7, R22.2, U5.B/Z
- net -TX: now also J2.1, J4.1, R9.2, U2.B/Z; no longer J3.1, J5.1, R2.2, U1.B/Z
- net 0V: now also C10.2, C11.2, C12.-, C16.2, J2.4, J2.5, J4.4, J4.5, J6.9, J7.2, J7.3, J8.6, J9.GND, R10.1, R21.1, R29.2, R31.2, R40.2, U1E.I, U1F.I, U1P.GND, U2.GND, U3P.GND, U6.GND, U7.0V@0, U7.0V@1, U8.GND; no longer C10.-, C12.2, J10.GND, J2.GND@0, J2.GND@1, J3.4, J3.5, J5.5, J6.4, J7.9, J8.2, J8.3, J9.6, R13.1, R21.2, R23.2, R3.1, R32.2, U1.GND, U2P.GND, U3.GND, U6.0V@0, U6.0V@1, U7.GND
- net DTR_!RE: now also R21.2, U4.!RE, U7.(OC0A)PD6; no longer R13.2, U3.!RE, U6.(OC0A)PD6
- net DTR_DE: now also R25.2, U7.PD7; no longer R17.2, U6.PD7
- net DTR_RXD: now also R26.2, U7.(RXD)PD0; no longer R18.2, U6.(RXD)PD0
- net DTR_TXD: now also R24.2, U4.DI, U7.(TXD)PD1; no longer R16.2, U3.DI, U6.(TXD)PD1
- net HOST_!CTS: now also R8.1, U1A.I, U7.(A0/MISO1)PC0; no longer J1.!CE12!/BCM16, U6.(A0/MISO1)PC0
- net HOST_!DSR: now also U7.(A1/SCK1)PC1; no longer U6.(A1/SCK1)PC1
- net HOST_!DTR: now also U7.(INT0/OC3B)PD2; no longer U6.(INT0/OC3B)PD2
- net HOST_!RTS: now also R5.1, U1D.O, U7.(INT1/OC2B)PD3; no longer C11.1, J1.BCM17/!CE11!, U6.(INT1/OC2B)PD3
- net HOST_MISO: now also R15.2, U3B.O; no longer R9.2, U2B.O
- net HOST_MOSI: now also U3E.I; no longer U2E.I
- net HOST_RX: now also R7.1, U1B.I, U2.RO; no longer J1.RXD/BCM15, R4.1, U1.RO
- net HOST_SCK: now also U3F.I; no longer U2F.I
- net HOST_TX: now also R32.1, R6.1, U1C.O, U6.DI; no longer J1.TXD/BCM14, R24.1, U5.DI
- net ICP1: now also R43.2, U7.(ICP1)PB0; no longer R33.2, U6.(ICP1)PB0
- net IOREF: now also J8.2, R16.1, R17.1, R27.1; no longer J9.2, R10.1, R11.1, R19.1
- net LED_BUILTIN: now also U7.(OC1A)PB1; no longer U6.(OC1A)PB1
- net MGR_!RESET: now also J9.!RESET, R35.1, U7.!RESET; no longer J10.!RESET, R27.1, U6.!RESET
- net MGR_!SS!: now also R38.1, U7.(!SS!/OC1B)PB2; no longer R30.1, U6.(!SS!/OC1B)PB2
- net MGR_AREF: now also C14.1, U7.AREF; no longer C12.1, U6.AREF
- net MGR_MISO: now also J9.MISO, U7.(MISO/RX1)PB4; no longer J10.MISO, U6.(MISO/RX1)PB4
- net MGR_MOSI: now also J9.MOSI, U7.(MOSI/TX1)PB3; no longer J10.MOSI, U6.(MOSI/TX1)PB3
- net MGR_SCK: now also J9.SCK, U7.(SCK)PB5; no longer J10.SCK, U6.(SCK)PB5
- net MISO: now also J8.1, U3B.I; no longer J9.1, U2B.I
- net MOSI: now also J8.4, R18.1; no longer J9.4, R11.2, U2E.O
- net N$10: now also R27.2, R33.2, U3C.O; no longer R19.2, R25.2, U2C.O
- net N$11: now also R34.2, U6.DE; no longer R26.2, U5.DE
- net N$15: now also R13.1; no longer R7.1
- net N$18: now also R11.1, U2.DE; no longer R5.1, U1.DE
- net N$19: now also R22.1, R26.1, U4.RO; no longer R14.1, R18.1, U3.RO
- net N$2: now also R38.2, U3D.I; no longer C11.2, R30.2, U2D.I
- net N$20: now also R25.1, U4.DE; no longer R17.1, U3.DE
- net N$22: now also R24.1; no longer R16.1
- net N$24: now also C11.1, U8.ADJ; no longer C9.1, U7.ADJ
- net N$25: now also R32.2; no longer R24.2
- net N$29: now also R45.2; no longer R34.2
- net NODE5V: now also J7.4, R39.2, U8.EN, U8.IN; no longer J8.4, U7.EN, U7.IN
- net RX: now also J3.3, R33.1; no longer J4.3, R25.1
- net RX_!RE: now also R31.1, U6.!RE, U7.(T0)PD4; no longer R23.1, U5.!RE, U6.(T0)PD4
- net RX_DE: now also R34.1, U7.(A3)PC3; no longer R26.1, U6.(A3)PC3
- net RX_RPU: now also R23.1, U3C.I, U6.RO; no longer R15.1, U2C.I, U5.RO
- net SCK: now also J8.3, R19.1; no longer J9.3, R10.2, U2F.O
- net SCL: now also J5.1, R37.1, U7.(A5/SCL0)PC5; no longer J6.1, R29.2
- net SDA: now also J5.2, R36.1, U7.(A4/SDA0)PC4; no longer J6.2, R28.2
- net SHUTDOWN: now also R44.1; no longer R33.1, S2.1, S2.2
- net TX: now also J3.4, R13.2, R14.2, U3A.I; no longer J4.4, R7.2, R8.2, U2A.I
- net TX_!RE: now also R10.2, U2.!RE, U7.(A2)PC2; no longer R3.2, U1.!RE, U6.(A2)PC2
- net TX_DE: now also R11.2, U7.(T1/OC0B)PD5; no longer R5.2, U6.(T1/OC0B)PD5
- net TX_RPU: now also R12.2, U2.DI, U3A.O; no longer R6.2, U1.DI, U2A.O
- net VIN: now also C4.1, J7.1, U5.VIN; no longer J8.1, R20.1, U4.VIN
- net XTAL1: now also C15.1, U7.XTAL1; no longer C13.1, U6.XTAL1
- net XTAL2: now also C16.1, U7.XTAL2; no longer C14.1, U6.XTAL2
Other:
- note added: "* 328PB IS NOT USED YET"
- note added: "2/7/17"
- note added: "5V FROM MCU NODE USED TO PWR RPU_BUS i.e. RPUpi WORKS LIKE RPUadpt W/O PI OR IF VIN POWER IS OFF"
- note added: "AVR AT 5V SEE 3V3 JUST FINE."
- note added: "CRYSTAL: ECS-120-20-3X-TR 12MHZ +/- 30PPM STABILITY AND TOLERANCE CRYSTAL CAPACITORS: 15PF = 5PF + (20PF*20PF)/(20PF+20PF)"
- note added: "I2C TO MCU BOARD"
- note added: "IF THE 3V3PI IS OFF THE 74LVC07 OPEN DRAIN IS HI-Z."
- note added: "SERIAL/SPI 74LVC07 PI3V3 OPEN SPI, TX PULLUP, I2C"
- note added: "^2"
- note removed: "* 328PB IS NOT USED"
- note removed: "5V FROM MCU NODE USED TO PWR RPU_BUS i.e. RPUpi WORKS LIKE RPUadpt W/O PI OR IF VIN IS OFF"
- note removed: "CRYSTAL NOT USED: ECS-147.4-20-3X-TR 14.7456MHZ +/- 30PPM STABILITY AND TOLERANCE CRYSTAL CAPACITORS: 15PF = 5PF + (20PF*20PF)/(20PF+20PF)"
- note removed: "MEGA AVR HAVE A WEAK PULL UP BUT WILL SEE 3V3 JUST FINE. ONE DANGER IS IF THE PIN IS SET AS AN OUTPUT HIGH IT WILL KILL THE PI."
- note removed: "PI AND OPENOCD https://learn.adafruit.com/programming-microcontrollers-using-openocd-on-raspberry-pi"
- note removed: "R4 NEEDED WHEN TX_!RE! IS USED TO BLOCK TX PAIR FROM HOST"
- moved on the sheet: C11, C13, C14, C15, C3, C4, C6, C7, C8, C9, J6, R1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
